File: PCB for desk pet/PCB for desk pet.kicad_sch (KiCad schematic)
At the start: 0 parts

Commit message: schematic done
Parts:
- added BZ1: Buzzer, symbol Device:Buzzer
- added Display: Conn_01x07, symbol Connector_Generic:Conn_01x07
- added ESP-left, ESP-right: Conn_01x22, Connector_PinSocket_2.54mm:PinSocket_1x22_P2.54mm_Vertical, symbol Connector_Generic:Conn_01x22
- added J1, J3: Conn_01x02, symbol Connector_Generic:Conn_01x02
- added J2: Conn_01x04, symbol Connector_Generic:Conn_01x04
- added SW1: SW_SPDT, symbol Switch:SW_SPDT
- added SW2, SW3: SW_Push, symbol Switch:SW_Push
Connections:
- new net +3V3: Display.2 (Pin_2), ESP-left.3 (Pin_3)
- new net +5V: ESP-left.1 (Pin_1), SW1.2 (B)
- new net BTN_ACTION: ESP-left.5 (Pin_5), SW3.1
- new net BTN_MENU: ESP-left.4 (Pin_4), SW2.1
- new net BUZZER: BZ1.1 (+), ESP-right.18 (Pin_18)
- new net GND: BZ1.2 (-), Display.1 (Pin_1), ESP-left.2 (Pin_2), ESP-right.1 (Pin_1), J1.2 (Pin_2), J2.3 (Pin_3), J2.4 (Pin_4), J3.2 (Pin_2), SW2.2, SW3.2
- new net LCD_CS: Display.7 (Pin_7), ESP-right.12 (Pin_12)
- new net LCD_DC: Display.6 (Pin_6), ESP-right.13 (Pin_13)
- new net LCD_RES: Display.5 (Pin_5), ESP-right.14 (Pin_14)
- new net LCD_SCL: Display.3 (Pin_3), ESP-right.10 (Pin_10)
- new net LCD_SDA: Display.4 (Pin_4), ESP-right.11 (Pin_11)
- new net USB_5V: J1.1 (Pin_1)
- new net VBAT: J2.2 (Pin_2), J3.1 (Pin_1)
- new net V_UNSW: J2.1 (Pin_1), SW1.1 (A)
- no-connect marks 0 -> 34
