File: PCB for desk pet/PCB for desk pet.kicad_sch (KiCad schematic)
At the start: 10 parts, among them J1 Conn_01x02, J2 Conn_01x04, J3 Conn_01x02, SW1 SW_SPDT, SW2 SW_Push, SW3 SW_Push

Commit message: backup
Parts:
- BZ1: footprint (none) -> Buzzer_Beeper:Buzzer_12x9.5RM7.6
- Display1: footprint (none) -> Connector_PinSocket_2.54mm:PinSocket_1x07_P2.54mm_Vertical
- J1: footprint (none) -> Connector_PinHeader_2.54mm:PinHeader_1x02_P2.54mm_Vertical
- J2: footprint (none) -> Connector_PinHeader_2.54mm:PinHeader_1x04_P2.54mm_Vertical
- J3: footprint (none) -> Connector_JST:JST_PH_B2B-PH-K_1x02_P2.00mm_Vertical
- SW1: footprint (none) -> Connector_PinHeader_2.54mm:PinHeader_1x03_P2.54mm_Vertical
- SW2, SW3: footprint (none) -> Button_Switch_THT:SW_PUSH_6mm_H5mm
Connections:
- net +3V3: now also ESP-left1.1 (Pin_1); no longer ESP-left1.3 (Pin_3)
- net +5V: now also ESP-left1.21 (Pin_21); no longer ESP-left1.1 (Pin_1)
- net BUZZER: now also ESP-left1.11 (Pin_11); no longer ESP-right1.18 (Pin_18)
- net GND: now also ESP-left1.22 (Pin_22), ESP-right1.21 (Pin_21), ESP-right1.22 (Pin_22); no longer ESP-left1.2 (Pin_2)
- net LCD_CS: now also ESP-left1.18 (Pin_18); no longer ESP-right1.12 (Pin_12)
- net LCD_DC: now also ESP-left1.19 (Pin_19); no longer ESP-right1.13 (Pin_13)
- net LCD_RES: now also ESP-left1.20 (Pin_20); no longer ESP-right1.14 (Pin_14)
- net LCD_SCL: now also ESP-left1.16 (Pin_16); no longer ESP-right1.10 (Pin_10)
- net LCD_SDA: now also ESP-left1.17 (Pin_17); no longer ESP-right1.11 (Pin_11)
- net USB_5V: no longer names the net of J1.1 (Pin_1)
- no-connect marks 34 -> 32

Commit message: PCB done
Parts:
- removed J2: Conn_01x04, Connector_PinHeader_2.54mm:PinHeader_1x04_P2.54mm_Vertical, symbol Connector_Generic:Conn_01x04
- added J2, J4: Conn_01x02, Connector_PinHeader_2.54mm:PinHeader_1x02_P2.54mm_Vertical, symbol Connector_Generic:Conn_01x02
- SW1: footprint Connector_PinHeader_2.54mm:PinHeader_1x03_P2.54mm_Vertical -> extra:SW_Toggle_Blue_wSlots
Connections:
- net GND: now also J4.2 (Pin_2); no longer J3.2 (Pin_2)
- net V_UNSW: now also J4.1 (Pin_1)
- net VBAT renamed BAT+
- net BAT+: now also J2.1 (Pin_1)
- new net BAT-: J2.2 (Pin_2), J3.2 (Pin_2)
Other:
- moved on the sheet: BZ1, Display1, J1, J3
