File: PCB for desk pet/_restore_backup_2026-10-06T23-20-22-108/PCB for desk pet.kicad_sch (KiCad schematic)
At the start: 10 parts, among them J1 Conn_01x02, J2 Conn_01x04, J3 Conn_01x02, SW1 SW_SPDT, SW2 SW_Push, SW3 SW_Push

Commit message: schematic
Parts:
- renumbered Display1 to Display, ESP-left1 to ESP-left, ESP-right1 to ESP-right
Other:
- moved on the sheet: BZ1, J1, J2, J3, SW1, SW2, SW3
